Commit message: Refactor URDF file for robot arm structure

File: simulation/4dofarm.urdf (robot description, URDF)
Before this commit: robot robot_arm_5dof, 11 links, 10 joints
Links:
- link base_link: geometry collision box size=0.12 0.12 0.008; visual mesh filename=package://4dofarm/meshes/base.stl scale=0.001 0.001 0.001
- link base_servo: geometry collision box size=0.0407 0.0197 0.0429; visual mesh filename=package://4dofarm/meshes/mg996r.stl scale=0.001 0.001 0.001
- link elbow_servo: geometry collision box size=0.023 0.0125 0.022; visual mesh filename=package://4dofarm/meshes/sg90.stl scale=0.001 0.001 0.001
- link end_servo: geometry collision box size=0.023 0.0125 0.022; visual mesh filename=package://4dofarm/meshes/sg90.stl scale=0.001 0.001 0.001
- link link1: geometry collision box size=0.11 0.018 0.004; visual mesh filename=package://4dofarm/meshes/link1.stl scale=0.001 0.001 0.001
- link link2: geometry collision box size=0.09 0.018 0.004; visual mesh filename=package://4dofarm/meshes/link2.stl scale=0.001 0.001 0.001
- link link3: geometry collision box size=0.055 0.014 0.004; visual box size=0.055 0.014 0.004
- link shoulder_servo: geometry collision box size=0.023 0.0125 0.022; visual mesh filename=package://4dofarm/meshes/sg90.stl scale=0.001 0.001 0.001
- link tool_link: geometry collision box size=0.070 0.014 0.004; visual box size=0.070 0.014 0.004
- link wrist_servo: geometry collision box size=0.023 0.0125 0.022; visual mesh filename=package://4dofarm/meshes/sg90.stl scale=0.001 0.001 0.001
Joints:
- joint base_mount: origin xyz=0 0 0.024 -> xyz=0 0 0.02545
- joint base_yaw: origin xyz=0 0 0.044 -> xyz=0 0 0.035
- joint elbow_pitch: origin xyz=0 0 0.028 -> xyz=0 0 0.011
- joint end_yaw: origin xyz=0 0 0.028 -> xyz=0 0 0.012
- joint link3_mount: origin xyz=0.012 0 0.028 -> xyz=0.012 0 0
- joint shoulder_pitch: origin xyz=0 0 0.028 -> xyz=0 0 0.012
